File: PCB/jlink-adapter.kicad_pcb (KiCad board)
At the start: 4 copper layers, 0 parts

Commit message: V1 PCB.
Parts:
- added D1: Yellow, LED_SMD:LED_1206_3216Metric_Pad1.42x1.75mm_HandSolder, F.Cu at (53.0, 53.5)
- added D2: Red, LED_SMD:LED_1206_3216Metric_Pad1.42x1.75mm_HandSolder, F.Cu at (53.0, 56.0)
- added D3: D5V0L1B2WS-7, Diode_SMD:D_SOD-323_HandSoldering, F.Cu at (51.3, 60.8)
- added J1: Conn_02x10_Odd_Even, Connector_PinHeader_2.54mm:PinHeader_2x10_P2.54mm_Horizontal, F.Cu at (61.5, 51.9)
- added J2: Conn_02x05_Odd_Even, JLink-adapter:PinHeader_2x05_P1.27mm_Vertical_comb_SMT_TH, F.Cu at (54.1, 67.8)
- added J3: Conn_02x05_Odd_Even, Connector_PinHeader_1.27mm:PinHeader_2x05_P1.27mm_Vertical_SMD, F.Cu at (54.8, 70.3)
- added JP1: Jumper_2_Bridged, Jumper:SolderJumper-2_P1.3mm_Bridged_RoundedPad1.0x1.5mm, B.Cu at (56.6, 53.0)
- added JP2: Jumper_2_Bridged, Jumper:SolderJumper-2_P1.3mm_Bridged_RoundedPad1.0x1.5mm, B.Cu at (56.6, 56.0)
- added Q1: BSS123TA, Package_TO_SOT_SMD:SOT-23, F.Cu at (54.9, 60.5)
- added R1: 1k, Resistor_SMD:R_0402_1005Metric_Pad0.72x0.64mm_HandSolder, F.Cu at (59.0, 53.0)
- added R2: 1k, Resistor_SMD:R_0402_1005Metric_Pad0.72x0.64mm_HandSolder, F.Cu at (59.0, 56.5)
- added R3: 100, Resistor_SMD:R_0402_1005Metric_Pad0.72x0.64mm_HandSolder, F.Cu at (59.1, 60.0)
- added R4: 100k, Resistor_SMD:R_0402_1005Metric_Pad0.72x0.64mm_HandSolder, F.Cu at (59.1, 63.5)
Routing:
- net GND: track 0.00 -> 60.9 mm, vias 0 -> 2
- net +5V: track 0.00 -> 24.6 mm
- net /VTREF: track 0.00 -> 19.8 mm, vias 0 -> 1
- net Net-(D3-A2): track 0.00 -> 12.2 mm, vias 0 -> 2
- net /SWDIO: track 0.00 -> 10.9 mm
- net /SWCLK: track 0.00 -> 10.1 mm
- net Net-(D2-K): track 0.00 -> 7.12 mm
- net /SWO: track 0.00 -> 6.04 mm
- net /RESET: track 0.00 -> 6.04 mm
- net Net-(D1-A): track 0.00 -> 4.93 mm
- net Net-(D2-A): track 0.00 -> 4.53 mm
- net Net-(JP2-A): track 0.00 -> 2.67 mm, vias 0 -> 1
- net Net-(JP1-A): track 0.00 -> 2.46 mm, vias 0 -> 1
Other:
- board outline added: 15.5 x 27 mm
- copper layers 4 -> 2
- board text added: "JLink Adapter SWD"
- board text added: "MCU_PWR"
- board text added: "SKEC V1"
- board text added: "USB_PWR"
- board text removed: "In1, [Description]"
- board text removed: "In2, [Description]"
