File: PCB/jlink-adapter.kicad_sch (KiCad schematic)
At the start: 0 parts

Commit message: V1 PCB.
Parts:
- added D1: Yellow, LED_SMD:LED_1206_3216Metric_Pad1.42x1.75mm_HandSolder, symbol Device:LED
- added D2: Red, LED_SMD:LED_1206_3216Metric_Pad1.42x1.75mm_HandSolder, symbol Device:LED
- added D3: D5V0L1B2WS-7, Diode_SMD:D_SOD-323_HandSoldering, symbol Device:D_TVS_Filled
- added J1: Conn_02x10_Odd_Even, Connector_PinHeader_2.54mm:PinHeader_2x10_P2.54mm_Horizontal, symbol Connector_Generic:Conn_02x10_Odd_Even
- added J2: Conn_02x05_Odd_Even, JLink-adapter:PinHeader_2x05_P1.27mm_Vertical_comb_SMT_TH, symbol Connector_Generic:Conn_02x05_Odd_Even
- added J3: Conn_02x05_Odd_Even, Connector_PinHeader_1.27mm:PinHeader_2x05_P1.27mm_Vertical_SMD, symbol Connector_Generic:Conn_02x05_Odd_Even
- added JP1, JP2: Jumper_2_Bridged, Jumper:SolderJumper-2_P1.3mm_Bridged_RoundedPad1.0x1.5mm, symbol Jumper:Jumper_2_Bridged
- added Q1: BSS123TA, Package_TO_SOT_SMD:SOT-23, symbol Device:Q_NMOS_GSD
- added R1, R2: 1k, Resistor_SMD:R_0402_1005Metric_Pad0.72x0.64mm_HandSolder, symbol Device:R_Small
- added R3: 100, Resistor_SMD:R_0402_1005Metric_Pad0.72x0.64mm_HandSolder, symbol Device:R_Small
- added R4: 100k, Resistor_SMD:R_0402_1005Metric_Pad0.72x0.64mm_HandSolder, symbol Device:R_Small
Connections:
- new net: JP2.1 (A), R2.1
- new net: D2.2 (A), R2.2
- new net: D2.1 (K), Q1.3 (D)
- new net: JP1.1 (A), R1.1
- new net: D3.2 (A2), Q1.1 (G), R3.2, R4.1
- new net: D1.2 (A), R1.2
- new net +5V: J1.19 (Pin_19), JP1.2 (B), JP2.2 (B)
- new net GND: D1.1 (K), D3.1 (A1), J1.10 (Pin_10), J1.12 (Pin_12), J1.4 (Pin_4), J1.6 (Pin_6), J1.8 (Pin_8), J2.3 (Pin_3), J2.5 (Pin_5), J2.9 (Pin_9), J3.3 (Pin_3), J3.5 (Pin_5), J3.9 (Pin_9), Q1.2 (S), R4.2
- new net NC_7: J2.7 (Pin_7), J3.7 (Pin_7)
- new net NC_8: J2.8 (Pin_8), J3.8 (Pin_8)
- new net RESET: J1.15 (Pin_15), J2.10 (Pin_10), J3.10 (Pin_10)
- new net SWCLK: J1.9 (Pin_9), J2.4 (Pin_4), J3.4 (Pin_4)
- new net SWDIO: J1.7 (Pin_7), J2.2 (Pin_2), J3.2 (Pin_2)
- new net SWO: J1.13 (Pin_13), J2.6 (Pin_6), J3.6 (Pin_6)
- new net VTREF: J1.1 (Pin_1), J2.1 (Pin_1), J3.1 (Pin_1), R3.1
- no-connect marks 0 -> 9
Other:
- note added: "NC_7 and NC_8 are No-Connects. They are there to prevent DRC errors in the PCB."
