File: Breadboard Power Supply Adapter/Breadboard Power Supply Adapter.kicad_pcb (KiCad board)
At the start: 2 copper layers, 52.1 x 15.2 mm, 18 parts, among them J1 Conn_02x03_Odd_Even, J2 Conn_02x03_Odd_Even, J3 Conn_01x02, J4 Conn_01x02

Commit message: Made V2 Breadboard Power Supply Adapter
Removed several redundant test points.  Re-using the Banana jack pads is
sufficient for Keystone and wires.

Added 3-pin regulator footprint, along with output pin.  Could be used
for secondary voltage supply or reference regulator.
Parts:
- removed TP10, TP7, TP8, TP9: Test Loop, TestPoint:TestPoint_Keystone_5010-5014_Multipurpose
- removed TP3, TP5: Solder Point, Connector_Wire:SolderWire-2sqmm_1x01_D2mm_OD3.9mm
- removed TP4, TP6: Solder Point, Connector_Wire:SolderWire-0.75sqmm_1x01_D1.25mm_OD3.5mm
- added J5: Conn_01x03, Connector_PinHeader_2.54mm:PinHeader_1x03_P2.54mm_Vertical, F.Cu at (68.5, 56.0)
- added J6: Conn_01x01, TestPoint:TestPoint_Keystone_5010-5014_Multipurpose, F.Cu at (80.3, 56.0)
- REF**: moved to F.Cu
- moved REF** 0.60 mm to (69.0, 46.4), turned to 0 degrees
- moved JP1 0.49 mm to (74.3, 45.2)
- moved D1 0.25 mm to (74.3, 50.8)
Routing:
- net /VREF: track 0.00 -> 6.76 mm
Other:
- board text added: "BB PowerSupply Adapter"
- board text added: "V2"
- board text added: "VREF"
- board text removed: "BB Power Supply Adapter"
- board text removed: "V1"
