File: cr2032_battery_load_tester/CR2032_battery_load_tester.kicad_sch (KiCad schematic)
At the start: 0 parts

Commit message: V1.0 of 2032 PCB
Parts:
- added BT1: Battery_Cell, Battery:BatteryHolder_Keystone_3034_1x20mm, symbol Device:Battery_Cell
- added R1: 100, Resistor_SMD:R_0603_1608Metric_Pad0.98x0.95mm_HandSolder, symbol Device:R_Small
- added SW6: SW_Push, Button_Switch_SMD:SW_Push_1P1T-SH_NO_CK_KMR2xxG, symbol Switch:SW_Push
- added TP1, TP2: TestPoint, TestPoint:TestPoint_Keystone_5010-5014_Multipurpose, symbol Connector:TestPoint
Connections:
- new net: R1.2, SW6.2
- new net +BATT: BT1.1 (+), R1.1, TP1.1
- new net GND: BT1.2 (-), SW6.1, TP2.1

Commit message: CR2032 Checkpoint, changing computers
Parts:
- added R2: 1k, Resistor_SMD:R_0603_1608Metric_Pad0.98x0.95mm_HandSolder, symbol Device:R_Small
- added SW6: SW_Push, Button_Switch_SMD:SW_Push_1P1T-SH_NO_CK_KMR2xxG, symbol Switch:SW_Push
Connections:
- net +BATT: now also R2.1
- net GND: now also SW6.1
- new net: R2.2, SW6.2
Other:
- moved on the sheet: TP1, TP2
Changed lines of the file:
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@@
     (company "SK Electronics Consulting")
   )
+  (junction (at 110.49 102.87) (diameter 0) (color 0 0 0 0)
+  )
   (junction (at 81.28 82.55) (diameter 0) (color 0 0 0 0)
   )
+  (junction (at 110.49 81.28) (diameter 0) (color 0 0 0 0)
+  )
   (junction (at 81.28 101.6) (diameter 0) (color 0 0 0 0)
   )
@@
     (stroke (width 0) (type default))
   )
+  (wire (pts (xy 110.49 88.9) (xy 110.49 91.44))
+    (stroke (width 0) (type default))
+  )
   (wire (pts (xy 96.52 81.28) (xy 96.52 83.82))
     (stroke (width 0) (type default))
@@
     (stroke (width 0) (type default))
   )
+  (wire (pts (xy 110.49 101.6) (xy 110.49 102.87))
+    (stroke (width 0) (type default))
+  )
+  (wire (pts (xy 110.49 81.28) (xy 110.49 83.82))
+    (stroke (width 0) (type default))
+  )
   (wire (pts (xy 81.28 81.28) (xy 96.52 81.28))
     (stroke (width 0) (type default))
   )
+  (wire (pts (xy 110.49 102.87) (xy 121.92 102.87))
+    (stroke (width 0) (type default))
+  )
   (wire (pts (xy 81.28 101.6) (xy 81.28 102.87))
     (stroke (width 0) (type default))
@@
     (stroke (width 0) (type default))
   )
-  (wire (pts (xy 96.52 81.28) (xy 101.6 81.28))
+  (wire (pts (xy 96.52 81.28) (xy 110.49 81.28))
     (stroke (width 0) (type default))
   )
@@
     (stroke (width 0) (type default))
   )
-  (wire (pts (xy 96.52 102.87) (xy 101.6 102.87))
+  (wire (pts (xy 96.52 102.87) (xy 110.49 102.87))
     (stroke (width 0) (type default))
   )
@@
   )
   (wire (pts (xy 81.28 81.28) (xy 81.28 82.55))
+    (stroke (width 0) (type default))
+  )
+  (wire (pts (xy 110.49 81.28) (xy 121.92 81.28))
     (stroke (width 0) (type default))
   )
@@
     )
   )
+  (symbol (lib_id "Switch:SW_Push") (at 110.49 96.52 270) (mirror x) (unit 1)
+    (in_bom yes) (on_board yes) (dnp no)
+    (property "Reference" "SW6" (at 118.11 96.52 90)
+      (effects (font (size 1.27 1.27)) (justify right))
+    )
+    (property "Value" "SW_Push" (at 109.22 97.79 90)
+      (effects (font (size 1.27 1.27)) (justify right) hide)
+    )
+    (property "Footprint" "Button_Switch_SMD:SW_Push_1P1T-SH_NO_CK_KMR2xxG" (at 115.57 96.52 0)
+      (effects (font (size 1.27 1.27)) hide)
+    )
+    (property "Datasheet" "~" (at 115.57 96.52 0)
+      (effects (font (size 1.27 1.27)) hide)
+    )
+    (property "Digikey PN" "401-1427-1-ND" (at 110.49 96.52 0)
+      (effects (font (size 1.27 1.27)) hide)
+    )
+    (property "MPN" "KMR221GLFS" (at 110.49 96.52 0)
+      (effects (font (size 1.27 1.27)) hide)
+    )
+    (property "URL" "https://www.digikey.com/en/products/detail/c-k/KMR221GLFS/550472" (at 110.49 96.52 0)
+      (effects (font (size 1.27 1.27)) hide)
+    )
+    (property "Mfg" "C&K" (at 110.49 96.52 0)
+      (effects (font (size 1.27 1.27)) hide)
+    )
+    (pin "1")
+    (pin "2")
+    (instances
+      (project "jamystor_pcb01"
+        (path "/105984c4-9bf7-480f-bc68-92d2719cc761/d6dc1cc0-5ab2-4a5d-b92a-0865cb26ede6"
+          (reference "SW6") (unit 1)
+        )
+      )
+      (project "CR2032_battery_load_tester"
+        (path "/c4b4938f-57db-4256-8168-815a3371e956"
+          (reference "SW2") (unit 1)
+        )
+      )
+    )
+  )
   (symbol (lib_id "power:GND") (at 81.28 104.14 0) (unit 1)
     (in_bom yes) (on_board yes) (dnp no) (fields_autoplaced)
@@
         (path "/c4b4938f-57db-4256-8168-815a3371e956"
           (reference "#PWR01") (unit 1)
+        )
+      )
+    )
+  )
+  (symbol (lib_id "Device:R_Small") (at 110.49 86.36 0) (unit 1)
+    (in_bom yes) (on_board yes) (dnp no) (fields_autoplaced)
+    (property "Reference" "R2" (at 113.03 85.09 0)
+      (effects (font (size 1.27 1.27)) (justify left))
+    )
+    (property "Value" "1k" (at 113.03 87.63 0)
+      (effects (font (size 1.27 1.27)) (justify left))
+    )
+    (property "Footprint" "Resistor_SMD:R_0603_1608Metric_Pad0.98x0.95mm_HandSolder" (at 110.49 86.36 0)
+      (effects (font (size 1.27 1.27)) hide)
+    )
+    (property "Datasheet" "~" (at 110.49 86.36 0)
+      (effects (font (size 1.27 1.27)) hide)
+    )
+    (pin "1")
+    (pin "2")
+    (instances
+      (project "CR2032_battery_load_tester"
+        (path "/c4b4938f-57db-4256-8168-815a3371e956"
+          (reference "R2") (unit 1)
         )
       )
@@
     )
   )
-  (symbol (lib_id "Connector:TestPoint") (at 101.6 81.28 270) (unit 1)
-    (in_bom yes) (on_board yes) (dnp no) (fields_autoplaced)
-    (property "Reference" "TP1" (at 106.68 81.28 90)
-      (effects (font (size 1.27 1.27)) (justify left))
-    )
-    (property "Value" "TestPoint" (at 106.68 82.55 90)
+  (symbol (lib_id "Connector:TestPoint") (at 121.92 81.28 270) (unit 1)
+    (in_bom yes) (on_board yes) (dnp no) (fields_autoplaced)
+    (property "Reference" "TP1" (at 127 81.28 90)
+      (effects (font (size 1.27 1.27)) (justify left))
+    )
+    (property "Value" "TestPoint" (at 127 82.55 90)
       (effects (font (size 1.27 1.27)) (justify left) hide)
     )
-    (property "Footprint" "TestPoint:TestPoint_Keystone_5010-5014_Multipurpose" (at 101.6 86.36 0)
-      (effects (font (size 1.27 1.27)) hide)
-    )
-    (property "Datasheet" "~" (at 101.6 86.36 0)
-      (effects (font (size 1.27 1.27)) hide)
-    )
-    (property "Digikey PN" "36-5010-ND" (at 101.6 81.28 0)
-      (effects (font (size 1.27 1.27)) hide)
-    )
-    (property "MPN" "5010" (at 101.6 81.28 0)
-      (effects (font (size 1.27 1.27)) hide)
-    )
-    (property "Mfg" "Keystone" (at 101.6 81.28 0)
-      (effects (font (size 1.27 1.27)) hide)
-    )
-    (property "URL" "https://www.digikey.com/en/products/detail/keystone-electronics/5010/255332?s=N4IgTCBcDaINYFMCeBnALgewHYIAQFYAGARkJAF0BfIA" (at 101.6 81.28 0)
+    (property "Footprint" "TestPoint:TestPoint_Keystone_5010-5014_Multipurpose" (at 121.92 86.36 0)
+      (effects (font (size 1.27 1.27)) hide)
+    )
+    (property "Datasheet" "~" (at 121.92 86.36 0)
+      (effects (font (size 1.27 1.27)) hide)
+    )
+    (property "Digikey PN" "36-5010-ND" (at 121.92 81.28 0)
+      (effects (font (size 1.27 1.27)) hide)
+    )
+    (property "MPN" "5010" (at 121.92 81.28 0)
+      (effects (font (size 1.27 1.27)) hide)
+    )
+    (property "Mfg" "Keystone" (at 121.92 81.28 0)
+      (effects (font (size 1.27 1.27)) hide)
+    )
+    (property "URL" "https://www.digikey.com/en/products/detail/keystone-electronics/5010/255332?s=N4IgTCBcDaINYFMCeBnALgewHYIAQFYAGARkJAF0BfIA" (at 121.92 81.28 0)
       (effects (font (size 1.27 1.27)) hide)
     )
@@
     )
   )
-  (symbol (lib_id "Connector:TestPoint") (at 101.6 102.87 270) (unit 1)
-    (in_bom yes) (on_board yes) (dnp no) (fields_autoplaced)
-    (property "Reference" "TP2" (at 106.68 102.87 90)
-      (effects (font (size 1.27 1.27)) (justify left))
-    )
-    (property "Value" "TestPoint" (at 106.68 104.14 90)
+  (symbol (lib_id "Connector:TestPoint") (at 121.92 102.87 270) (unit 1)
+    (in_bom yes) (on_board yes) (dnp no) (fields_autoplaced)
+    (property "Reference" "TP2" (at 127 102.87 90)
+      (effects (font (size 1.27 1.27)) (justify left))
+    )
+    (property "Value" "TestPoint" (at 127 104.14 90)
       (effects (font (size 1.27 1.27)) (justify left) hide)
     )
-    (property "Footprint" "TestPoint:TestPoint_Keystone_5010-5014_Multipurpose" (at 101.6 107.95 0)
-      (effects (font (size 1.27 1.27)) hide)
-    )
-    (property "Datasheet" "~" (at 101.6 107.95 0)
-      (effects (font (size 1.27 1.27)) hide)
-    )
-    (property "Digikey PN" "36-5010-ND" (at 101.6 102.87 0)
-      (effects (font (size 1.27 1.27)) hide)
-    )
-    (property "MPN" "5010" (at 101.6 102.87 0)
-      (effects (font (size 1.27 1.27)) hide)
-    )
-    (property "Mfg" "Keystone" (at 101.6 102.87 0)
-      (effects (font (size 1.27 1.27)) hide)
-    )
-    (property "URL" "https://www.digikey.com/en/products/detail/keystone-electronics/5010/255332?s=N4IgTCBcDaINYFMCeBnALgewHYIAQFYAGARkJAF0BfIA" (at 101.6 102.87 0)
-      (effects (font (size 1.27 1.27)) hide)
-    )
+    (property "Footprint" "TestPoint:TestPoint_Keystone_5010-5014_Multipurpose" (at 121.92 107.95 0)
+      (effects (font (size 1.27 1.27)) hide)
+    )
+    (property "Datasheet" "~" (at 121.92 107.95 0)
+      (effects (font (size 1.27 1.27)) hide)
+    )
+    (property "Digikey PN" "36-5010-ND" (at 121.92 102.87 0)
+      (effects (font (size 1.27 1.27)) hide)
+    )
+    (property "MPN" "5010" (at 121.92 102.87 0)
+      (effects (font (size 1.27 1.27)) hide)
+    )
+    (property "Mfg" "Keystone" (at 121.92 102.87 0)
+      (effects (font (size 1.27 1.27)) hide)
+    )
+    (property "URL" "https://www.digikey.com/en/products/detail/keystone-electronics/5010/255332?s=N4IgTCBcDaINYFMCeBnALgewHYIAQFYAGARkJAF0BfIA" (at 121.92 102.87 0)
+      (effects (font (size 1.27 1.27)) hide)
+    )
