File: SAO_tree_ornament/SAO_tree_ornament.kicad_pcb (KiCad board)
At the start: 4 copper layers, 30 x 40.5 mm, 23 parts, among them J1 USB_C_Receptacle_USB2.0_16P, J2 Conn_02x03_Odd_Even, J3 Conn_01x02, J4 Conn_01x02, J5 Conn_QWIIC_Vertical, J6 Conn_ARM_SWD_TagConnect_TC203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, U1 HUSB238, U2 LMR51430, U4 MSPM0C110xSDSG

Commit message: Update SAO Connector on badge
Parts:
- J2: footprint Connector_PinSocket_2.54mm:PinSocket_2x03_P2.54mm_Vertical -> SKEC_Footprints:SAO_Connector_Badge
- moved J2 2.84 mm to (50.0, 81.2)
