File: Gridfinity-USB-hub/downstream_port.kicad_sch (KiCad schematic)
At the start: 5 parts, among them J3 USB_C_Receptacle_USB2.0_16P

Commit message: USB Hub Board as order submitted on 9/6
This might get rejected by JLC for via sizes.
Changed lines of the file:
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@@
 	(bus
 		(pts
-			(xy 153.67 92.71) (xy 152.4 92.71)
+			(xy 153.67 92.71) (xy 137.16 92.71)
 		)
 		(stroke
@@
 	(hierarchical_label "USB{USB}"
 		(shape input)
-		(at 152.4 92.71 180)
+		(at 137.16 92.71 180)
 		(effects
 			(font
@@
 		)
 	)
+	(netclass_flag ""
+		(length 2.54)
+		(shape round)
+		(at 138.43 92.71 0)
+		(fields_autoplaced yes)
+		(effects
+			(font
+				(size 1.27 1.27)
+			)
+			(justify left bottom)
+		)
+		(property "Netclass" "USB_DATA"
+			(at 139.1285 90.17 0)
+			(effects
+				(font
+					(size 1.27 1.27)
+				)
+				(justify left)
+			)
+		)
+		(property "Component Class" ""
+			(at -64.77 10.16 0)
+			(effects
+				(font
+					(size 1.27 1.27)
+					(italic yes)
+				)
+			)
+		)
+	)
