File: Gridfinity-USB-hub/downstream_port.kicad_sch (KiCad schematic)
At the start: 5 parts, among them J3 USB_C_Receptacle_USB2.0_16P

Commit message: V2 complete, ready for review and polish
Parts:
- R6, R7: value 56k -> 10k; JLCPCB Part No. C25796 -> (none)
Connections:
- net GND: now also J3.SH (SHIELD); no longer J3.S1 (SHIELD)
Changed lines of the file:
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@@
 			)
 		)
-		(property "Value" "56k"
+		(property "Value" "10k"
 			(at 153.67 83.8199 0)
 			(effects
@@
 			)
 		)
-		(property "JLCPCB Part No." "C25796"
+		(property "JLCPCB Part No." ""
+			(at 151.13 82.55 0)
+			(effects
+				(font
+					(size 1.27 1.27)
+				)
+				(hide yes)
+			)
+		)
+		(property "KLC_S4.2_VREGOUT" ""
 			(at 151.13 82.55 0)
 			(effects
@@
 			)
 		)
+		(property "Sim.Pins" "1=K 2=A"
+			(at 80.01 91.44 0)
+			(effects
+				(font
+					(size 1.27 1.27)
+				)
+				(hide yes)
+			)
+		)
 		(pin "1"
 		)
@@
 			)
 		)
-		(property "Value" "56k"
+		(property "Value" "10k"
 			(at 161.29 83.8199 0)
 			(effects
@@
 			)
 		)
-		(property "JLCPCB Part No." "C25796"
+		(property "JLCPCB Part No." ""
 			(at 158.75 82.55 0)
 			(effects
@@
 		(pin "B12"
 		)
-		(pin "S1"
+		(pin "SH"
 		)
 		(pin "B5"

Commit message: Add 3x channels of spare LEDs for general breadboard use, add silkscreen.  Ordered this version
Parts:
- R6, R7: JLCPCB Part No. (none) -> C60490; MPN (none) -> RC0402FR-0710KL
Other:
- company: (none) -> SK Electronics Consulting LLC
- title: (none) -> USB 2.0 Hub for Gridifinity
Changed lines of the file:
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@@
 	(generator_version "9.0")
 	(paper "A4")
+	(title_block
+		(title "USB 2.0 Hub for Gridifinity")
+		(date "2026-02-16")
+		(rev "2")
+		(company "SK Electronics Consulting LLC")
+	)
 	(text "Future Feature Ideas:\n1. Add a power monitor to each channel\n2. Jumpers to adjust R_{p} values\n"
 		(exclude_from_sim no)
@@
 			)
 		)
-		(property "JLCPCB Part No." ""
+		(property "JLCPCB Part No." "C60490"
 			(at 151.13 82.55 0)
 			(effects
@@
 		)
 		(property "KLC_S4.2_VREGOUT" ""
+			(at 151.13 82.55 0)
+			(effects
+				(font
+					(size 1.27 1.27)
+				)
+				(hide yes)
+			)
+		)
+		(property "MPN" "RC0402FR-0710KL"
 			(at 151.13 82.55 0)
 			(effects
@@
 			)
 		)
-		(property "JLCPCB Part No." ""
+		(property "JLCPCB Part No." "C60490"
 			(at 158.75 82.55 0)
 			(effects
+				(font
+					(size 1.27 1.27)
+				)
+				(hide yes)
+			)
+		)
+		(property "MPN" "RC0402FR-0710KL"
+			(at 158.75 82.55 0)
+			(effects
