File: Gridfinity-USB-hub/Gridfinity-USB-hub.kicad_pcb (KiCad board)
At the start: 4 copper layers, 40 x 40 mm, 57 parts, among them J1 USB_C_Receptacle_USB2.0_16P, J2 QWIIC, J3 USB_C_Receptacle_USB2.0_16P, J4 USB_C_Receptacle_USB2.0_16P, J5 USB_C_Receptacle_USB2.0_16P, J6 USB_C_Receptacle_USB2.0_16P, J7 Conn_ARM_SWD_TagConnect_TC203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, J8 Conn_02x05_Odd_Even, U1 CH334F, U2 CH334F, U3 FT2232HQ, U4 RP2040, U5 W25Q16JVSS, Y1 12MHz, Y2 12MHz

Commit message: V2 complete, ready for review and polish
Parts:
- added C10: 10u, Capacitor_SMD:C_0603_1608Metric, F.Cu at (73.1, 63.3)
- added C11: 0.1u, Capacitor_SMD:C_0402_1005Metric, F.Cu at (77.5, 67.5)
- added C12: 10u, Capacitor_SMD:C_0603_1608Metric, F.Cu at (78.9, 67.1)
- added C13: 10u, Capacitor_SMD:C_0603_1608Metric, F.Cu at (81.4, 69.9)
- added C14: 0.1u, Capacitor_SMD:C_0402_1005Metric, F.Cu at (81.3, 68.6)
- added C15: 0.1u, Capacitor_SMD:C_0402_1005Metric, F.Cu at (77.3, 75.9)
- added C16: 12pF, Capacitor_SMD:C_0402_1005Metric, F.Cu at (80.7, 73.5)
- added C17: 12pF, Capacitor_SMD:C_0402_1005Metric, F.Cu at (78.7, 70.8)
- added C18: 10u, Capacitor_SMD:C_0603_1608Metric, F.Cu at (63.2, 66.9)
- added C19: 0.1u, Capacitor_SMD:C_0402_1005Metric, F.Cu at (71.9, 63.3)
- added C20: 0.1u, Capacitor_SMD:C_0402_1005Metric, F.Cu at (63.8, 70.2)
- added C21: 0.1u, Capacitor_SMD:C_0402_1005Metric, F.Cu at (67.5, 75.6)
- added C22: 0.1u, Capacitor_SMD:C_0402_1005Metric, F.Cu at (65.4, 75.6)
- added C23: 0.1u, Capacitor_SMD:C_0402_1005Metric, F.Cu at (75.5, 74.0)
- added C24: 47u, Capacitor_SMD:C_1206_3216Metric, F.Cu at (83.6, 85.1)
- added C25: 0.1u, Capacitor_SMD:C_0402_1005Metric, F.Cu at (60.0, 74.8)
- added C26: 0.1u, Capacitor_SMD:C_0402_1005Metric, F.Cu at (86.1, 78.2)
- added C27: 0.1u, Capacitor_SMD:C_0402_1005Metric, F.Cu at (58.8, 75.8)
- added C28: 0.1u, Capacitor_SMD:C_0402_1005Metric, F.Cu at (88.0, 77.1)
- added C29: 0.1u, Capacitor_SMD:C_0402_1005Metric, F.Cu at (61.0, 79.2)
- added C30: 0.1u, Capacitor_SMD:C_0402_1005Metric, F.Cu at (83.8, 80.4)
- added C31: 47u, Capacitor_SMD:C_1206_3216Metric, F.Cu at (54.0, 79.8)
- added C32: 0.1u, Capacitor_SMD:C_0402_1005Metric, F.Cu at (102.8, 60.6)
- added C33: 0.1u, Capacitor_SMD:C_0402_1005Metric, F.Cu at (108.2, 60.5)
- added C9: 0.1u, Capacitor_SMD:C_0402_1005Metric, F.Cu at (70.3, 76.0)
- added D10: Green, LED_SMD:LED_0402_1005Metric, F.Cu at (66.5, 82.2)
- added FB1: FerriteBead_Small, Inductor_SMD:L_0402_1005Metric, F.Cu at (80.7, 67.3)
- added FB2: FerriteBead_Small, Inductor_SMD:L_0402_1005Metric, F.Cu at (81.2, 71.2)
- added J10: Conn_02x05_Odd_Even, Connector_PinHeader_2.54mm:PinHeader_2x05_P2.54mm_Vertical, F.Cu at (52.5, 64.9)
- added J11: Conn_01x02, Connector_PinSocket_2.54mm:PinSocket_1x02_P2.54mm_Vertical, F.Cu at (121.4, 66.5)
- added J12: Conn_01x02, Connector_PinSocket_2.54mm:PinSocket_1x02_P2.54mm_Vertical, F.Cu at (98.6, 57.7)
- added J9: Conn_02x05_Odd_Even, Connector_PinHeader_2.54mm:PinHeader_2x05_P2.54mm_Vertical, F.Cu at (75.1, 52.5)
- added JP5: Jumper_2_Small_Bridged, Jumper:SolderJumper-2_P1.3mm_Bridged2Bar_RoundedPad1.0x1.5mm, F.Cu at (102.8, 63.3)
- added R17: 12k, Resistor_SMD:R_0402_1005Metric, F.Cu at (79.9, 75.5)
- added R18: 2k, Resistor_SMD:R_0402_1005Metric, F.Cu at (73.5, 78.6)
- added R19: 12k, Resistor_SMD:R_0402_1005Metric, F.Cu at (77.5, 65.5)
- added R20: 10k, Resistor_SMD:R_0402_1005Metric, F.Cu at (73.5, 76.6)
- added R21: 1M, Resistor_SMD:R_0402_1005Metric, F.Cu at (76.6, 72.7)
- added R22: 10k, Resistor_SMD:R_0402_1005Metric, F.Cu at (81.6, 88.2)
- added R23: 10k, Resistor_SMD:R_0402_1005Metric, F.Cu at (70.0, 85.1)
- added R24: 78.7, Resistor_SMD:R_0402_1005Metric, F.Cu at (57.8, 75.8)
- added R25: 78.7, Resistor_SMD:R_0402_1005Metric, F.Cu at (60.4, 77.8)
- added R26: 78.7, Resistor_SMD:R_0402_1005Metric, F.Cu at (88.0, 76.1)
- added R27: 78.7, Resistor_SMD:R_0402_1005Metric, F.Cu at (83.4, 79.0)
- added R28: 5m, Resistor_SMD:R_1206_3216Metric, F.Cu at (81.2, 80.4)
- added R29: 78.7, Resistor_SMD:R_0402_1005Metric, F.Cu at (83.4, 81.8)
- added R30: 5m, Resistor_SMD:R_1206_3216Metric, F.Cu at (58.2, 79.2)
- added R31: 78.7, Resistor_SMD:R_0402_1005Metric, F.Cu at (60.3, 80.6)
- added R32: 10k, Resistor_SMD:R_0402_1005Metric, F.Cu at (57.6, 89.0)
- added R33: 10k, Resistor_SMD:R_0402_1005Metric, F.Cu at (62.6, 81.4)
- added R34: 10k, Resistor_SMD:R_0402_1005Metric, F.Cu at (91.0, 82.8)
- added R35: 10k, Resistor_SMD:R_0402_1005Metric, F.Cu at (87.5, 73.4)
- added U6: 93LCxxBxxOT, Package_TO_SOT_SMD:SOT-23-6, F.Cu at (76.7, 78.2)
- added U7: INA226, Package_SO:TSSOP-10_3x3mm_P0.5mm, F.Cu at (87.8, 80.5)
- added Y3: 12MHz, Crystal:Crystal_SMD_2520-4Pin_2.5x2.0mm, F.Cu at (78.7, 73.1)
- J7: value Conn_ARM_SWD_TagConnect_TC2030-NL -> USB_C_Receptacle_USB2.0_16P; footprint Connector:Tag-Connect_TC2030-IDC-NL_2x03_P1.27mm_Vertical -> Connector_USB:USB_C_Receptacle_G-Switch_GT-USB-7051x; moved to F.Cu
- J8: value Conn_02x05_Odd_Even -> USB_C_Receptacle_USB2.0_16P; footprint Connector_PinHeader_1.27mm:PinHeader_2x05_P1.27mm_Vertical -> Connector_USB:USB_C_Receptacle_G-Switch_GT-USB-7051x
- JP1, JP2, JP3, JP4: moved to F.Cu
- R10, R11, R12, R13, R6, R7, R8, R9: value 56k -> 10k
- U3: value FT2232HQ -> FT2232H-56Q; footprint Package_DFN_QFN:QFN-64-1EP_9x9mm_P0.5mm_EP4.35x4.35mm -> Package_DFN_QFN:QFN-56-1EP_8x8mm_P0.5mm_EP5.9x5.9mm
- U4: value RP2040 -> INA226; footprint Package_DFN_QFN:QFN-56-1EP_7x7mm_P0.4mm_EP3.2x3.2mm -> Package_SO:TSSOP-10_3x3mm_P0.5mm
- U5: value W25Q16JVSS -> AP2112K-3.3; footprint Package_DFN_QFN:DFN-8-1EP_3x2mm_P0.5mm_EP1.7x1.6mm -> Package_TO_SOT_SMD:SOT-23-5
- moved U5 76.8 mm to (105.6, 60.0), turned to 180 degrees
- moved D6 65.0 mm to (98.7, 70.0), turned to 90 degrees
- moved J7 63.7 mm to (76.0, 86.0)
- moved D5 61.2 mm to (103.6, 82.2), turned to 180 degrees
- moved TH1 60.7 mm to (118.2, 58.8), turned to 0 degrees
- moved R14 58.8 mm to (99.9, 70.0), turned to 90 degrees
- moved C8 56.4 mm to (93.8, 65.5), turned to 90 degrees
- moved R12 54.5 mm to (111.6, 87.1), turned to -90 degrees
- moved C7 54.4 mm to (92.0, 65.5), turned to 90 degrees
- moved J8 52.8 mm to (64.0, 86.0)
- moved R13 52.4 mm to (106.3, 82.1)
- moved D9 47.7 mm to (66.7, 64.4), turned to 180 degrees
- moved R5 47.2 mm to (110.7, 57.8)
- moved D1 46.9 mm to (113.1, 57.8)
- moved C3 45.9 mm to (122.6, 59.7)
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Connections:
- net /LED_MID.A renamed /LED2.A
- net /LED_MID.K renamed /LED3.A
- net /USB_Hub/Upstream.D+ renamed /USB_Hub0/Upstream.D+
- net /USB_Hub/Upstream.D- renamed /USB_Hub0/Upstream.D-
- D8 pad 1: /LED7.K -> /LED4.A
- D9 pad 1: /LED4.K -> /LED7.K
- D9 pad 2: /LED7.K -> /LED4.K
- J2 pad 3: /Serial_comms/SDA -> /SENSOR_I2C.SDA
- J2 pad 4: /Serial_comms/SCL -> /SENSOR_I2C.SCL
- U3 pad 1: GND -> /Serial_comms/EECS
- U3 pad 11: GND -> Net-(U3-~{RESET})
- U3 pad 12: unconnected-(U3-VCORE-Pad12) -> /Serial_comms/ADBUS0
- U3 pad 13: unconnected-(U3-TEST-Pad13) -> /Serial_comms/ADBUS1
- U3 pad 14: unconnected-(U3-~{RESET}-Pad14) -> /Serial_comms/ADBUS2
- U3 pad 15: GND -> /Serial_comms/ADBUS3
- U3 pad 16: unconnected-(U3-ADBUS0-Pad16) -> +3V3
- U3 pad 17: unconnected-(U3-ADBUS1-Pad17) -> /Serial_comms/ADBUS4
- U3 pad 18: unconnected-(U3-ADBUS2-Pad18) -> /Serial_comms/ADBUS5
- U3 pad 19: unconnected-(U3-ADBUS3-Pad19) -> /Serial_comms/ADBUS6
- U3 pad 2: unconnected-(U3-OSCI-Pad2) -> /Serial_comms/VCORE
- U3 pad 20: +3V3 -> /Serial_comms/ADBUS7
- U3 pad 21: unconnected-(U3-ADBUS4-Pad21) -> GND
- U3 pad 25: GND -> unconnected-(U3-ACBUS3-Pad25)
- U3 pad 3: unconnected-(U3-OSCO-Pad3) -> Net-(U3-OSCI)
- U3 pad 31: +3V3 -> /Serial_comms/VCORE
- U3 pad 32: unconnected-(U3-ACBUS5-Pad32) -> /Serial_comms/BDBUS0
- U3 pad 33: unconnected-(U3-ACBUS6-Pad33) -> /Serial_comms/BDBUS1
- U3 pad 34: unconnected-(U3-ACBUS7-Pad34) -> /Serial_comms/BDBUS2
- U3 pad 35: GND -> /Serial_comms/BDBUS3
- U3 pad 36: unconnected-(U3-~{SUSPEND}-Pad36) -> +3V3
- U3 pad 37: unconnected-(U3-VCORE-Pad37) -> /Serial_comms/BDBUS4
- U3 pad 38: unconnected-(U3-BDBUS0-Pad38) -> /Serial_comms/BDBUS5
- U3 pad 39: unconnected-(U3-BDBUS1-Pad39) -> /Serial_comms/BDBUS6
- U3 pad 4: unconnected-(U3-VPHY-Pad4) -> Net-(U3-OSCO)
- U3 pad 40: unconnected-(U3-BDBUS2-Pad40) -> /Serial_comms/BDBUS7
- U3 pad 41: unconnected-(U3-BDBUS3-Pad41) -> GND
- U3 pad 42: +3V3 -> unconnected-(U3-BCBUS0-Pad42)
- U3 pad 43: unconnected-(U3-BDBUS4-Pad43) -> /Serial_comms/VCORE
- U3 pad 44: unconnected-(U3-BDBUS5-Pad44) -> +3V3
- U3 pad 45: unconnected-(U3-BDBUS6-Pad45) -> GND
- U3 pad 47: GND -> unconnected-(U3-BCBUS2-Pad47)
- U3 pad 5: GND -> /Serial_comms/VPHY
- U3 pad 50: unconnected-(U3-VREGIN-Pad50) -> +3V3
- U3 pad 51: GND -> unconnected-(U3-BCBUS5-Pad51)
- U3 pad 55: unconnected-(U3-BCBUS4-Pad55) -> /Serial_comms/EEDATA
- U3 pad 56: +3V3 -> /Serial_comms/EECLK
- U3 pad 57: unconnected-(U3-BCBUS5-Pad57) -> GND
- U3 pad 6: unconnected-(U3-REF-Pad6) -> Net-(U3-REF)
- U3 pad 7: /USB6.D- -> /USB7.D-
- U3 pad 8: /USB6.D+ -> /USB7.D+
- U3 pad 9: unconnected-(U3-VPLL-Pad9) -> /Serial_comms/VPLL
- U4 pad 1: +3V3 -> GND
- U4 pad 10: +3V3 -> Net-(U4-Vin+)
- U4 pad 2: unconnected-(U4-GPIO0-Pad2) -> /SENSOR_I2C.SCL
- U4 pad 4: unconnected-(U4-GPIO2-Pad4) -> /SENSOR_I2C.SDA
- U4 pad 5: unconnected-(U4-GPIO3-Pad5) -> /SENSOR_I2C.SCL
- U4 pad 6: unconnected-(U4-GPIO4-Pad6) -> +3V3
- U4 pad 7: unconnected-(U4-GPIO5-Pad7) -> GND
- U4 pad 8: unconnected-(U4-GPIO6-Pad8) -> Net-(U4-Vbus)
- U4 pad 9: unconnected-(U4-GPIO7-Pad9) -> Net-(U4-Vin-)
- U5 pad 1: unconnected-(U5-~{CS}-Pad1) -> VBUS
- U5 pad 2: unconnected-(U5-DO/IO_{1}-Pad2) -> GND
- U5 pad 3: unconnected-(U5-~{WP}/IO_{2}-Pad3) -> VBUS
- U5 pad 5: unconnected-(U5-DI/IO_{0}-Pad5) -> Net-(J12-Pin_1)
- Y1 pad 1: Net-(U1-XI) -> Net-(U1-XO)
- Y1 pad 3: Net-(U1-XO) -> Net-(U1-XI)
- Y2 pad 1: Net-(U2-XI) -> Net-(U2-XO)
- Y2 pad 3: Net-(U2-XO) -> Net-(U2-XI)
Routing:
- net /LED4.K: track 0.00 -> 88.1 mm, vias 0 -> 5
- net GND: track 44.5 -> 132.1 mm, vias 8 -> 43
- net /LED2.A: track 3.23 -> 59.5 mm, vias 0 -> 4
- net /LED7.K: track 0.00 -> 54.4 mm, vias 0 -> 4
- net /SENSOR_I2C.SCL: track 0.00 -> 50.8 mm, vias 0 -> 2
- net /LED4.A: track 0.00 -> 50.6 mm, vias 0 -> 4
- net /USB6.D-: track 0.00 -> 41.4 mm, vias 0 -> 2
- net /USB6.D+: track 0.00 -> 40.7 mm, vias 0 -> 3
- net /SENSOR_I2C.SDA: track 0.00 -> 36.9 mm, vias 0 -> 2
- net /USB5.D-: track 0.00 -> 30.8 mm, vias 0 -> 2
- net /USB5.D+: track 0.00 -> 30.1 mm, vias 0 -> 3
- net +3V3: track 9.87 -> 35.6 mm, vias 1 -> 18
- net /USB_MID.D-: track 0.00 -> 23.5 mm, vias 0 -> 2
- net /USB_MID.D+: track 0.00 -> 23.5 mm, vias 0 -> 2
- net /Serial_comms/VCORE: track 0.00 -> 22.5 mm, vias 0 -> 3
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- added copper zone on In2.Cu, net +3V3
Other:
- board size 40 x 40 mm -> 82 x 40 mm
- board text removed: "Debug"

Commit message: Add 3x channels of spare LEDs for general breadboard use, add silkscreen.  Ordered this version
Parts:
- added D11: Green, LED_SMD:LED_0402_1005Metric, F.Cu at (79.6, 52.4)
- added D12: Green, LED_SMD:LED_0402_1005Metric, F.Cu at (85.8, 52.4)
- added D13: Green, LED_SMD:LED_0402_1005Metric, F.Cu at (92.1, 52.5)
- added J13: Conn_01x02, Connector_PinSocket_2.54mm:PinSocket_1x02_P2.54mm_Vertical, F.Cu at (82.1, 55.0)
- added J14: Conn_01x02, Connector_PinSocket_2.54mm:PinSocket_1x02_P2.54mm_Vertical, F.Cu at (88.3, 55.0)
- added J15: Conn_01x02, Connector_PinSocket_2.54mm:PinSocket_1x02_P2.54mm_Vertical, F.Cu at (94.5, 55.0)
- added JP6: Jumper_2_Small_Bridged, Jumper:SolderJumper-2_P1.3mm_Bridged2Bar_RoundedPad1.0x1.5mm, F.Cu at (79.4, 58.5)
- added JP7: Jumper_2_Small_Bridged, Jumper:SolderJumper-2_P1.3mm_Bridged2Bar_RoundedPad1.0x1.5mm, F.Cu at (85.6, 58.5)
- added JP8: Jumper_2_Small_Bridged, Jumper:SolderJumper-2_P1.3mm_Bridged2Bar_RoundedPad1.0x1.5mm, F.Cu at (91.8, 58.5)
- added R36: 2k, Resistor_SMD:R_0402_1005Metric, F.Cu at (81.8, 52.4)
- added R37: 2k, Resistor_SMD:R_0402_1005Metric, F.Cu at (88.0, 52.4)
- added R38: 2k, Resistor_SMD:R_0402_1005Metric, F.Cu at (94.4, 52.5)
- U6: value 93LCxxBxxOT -> 93LC56BxxOT
- moved JP2 0.75 mm to (93.6, 62.6), turned to 180 degrees
Connections:
- net /LED2.A renamed /LED_MID.A
- net /LED3.A renamed /LED_MID.K
Routing:
- net Net-(D12-K): track 0.00 -> 5.63 mm
- net Net-(D11-K): track 0.00 -> 5.63 mm
- net Net-(D13-K): track 0.00 -> 5.54 mm
- net Net-(J15-Pin_1): track 0.00 -> 2.73 mm
- net Net-(J14-Pin_1): track 0.00 -> 2.70 mm
- net Net-(J13-Pin_1): track 0.00 -> 2.70 mm
- net Net-(D13-A): track 0.00 -> 1.32 mm
- net Net-(D11-A): track 0.00 -> 1.21 mm
- net Net-(D12-A): track 0.00 -> 1.20 mm
- net GND: vias 43 -> 46
Other:
- board text added: "+3V3"
- board text added: "+5V"
- board text added: "GND"
