File: Gridfinity-USB-hub/Serial_comms.kicad_sch (KiCad schematic)
At the start: 3 parts, among them J2 QWIIC, U3 FT2232HQ

Commit message: V2 complete, ready for review and polish
Parts:
- removed J2: QWIIC, Connector_JST:JST_SH_BM04B-SRSS-TB_1x04-1MP_P1.00mm_Vertical, symbol SKEC_Symbols:Conn_QWIIC_Vertical
- removed U3: FT2232HQ, Package_DFN_QFN:QFN-64-1EP_9x9mm_P0.5mm_EP4.35x4.35mm, symbol Interface_USB:FT2232HQ
- added C10, C12, C13, C18: 10u, Capacitor_SMD:C_0603_1608Metric, symbol Device:C_Small
- added C11, C14, C15, C19, C20, C21, C22, C23, C9: 0.1u, Capacitor_SMD:C_0402_1005Metric, symbol Device:C_Small
- added C16, C17: 12pF, Capacitor_SMD:C_0402_1005Metric, symbol Device:C_Small
- added FB1, FB2: FerriteBead_Small, Inductor_SMD:L_0402_1005Metric, symbol Device:FerriteBead_Small
- added J10, J9: Conn_02x05_Odd_Even, Connector_PinHeader_2.54mm:PinHeader_2x05_P2.54mm_Vertical, symbol Connector_Generic:Conn_02x05_Odd_Even
- added R17, R19: 12k, Resistor_SMD:R_0402_1005Metric, symbol Device:R_Small
- added R18: 2k, Resistor_SMD:R_0402_1005Metric, symbol Device:R_Small
- added R20: 10k, Resistor_SMD:R_0402_1005Metric, symbol Device:R_Small
- added R21: 1M, Resistor_SMD:R_0402_1005Metric, symbol Device:R_Small
- added U3: FT2232H-56Q, Package_DFN_QFN:QFN-56-1EP_8x8mm_P0.5mm_EP5.9x5.9mm, symbol Interface_USB:FT2232H-56Q
- added U6: 93LCxxBxxOT, Package_TO_SOT_SMD:SOT-23-6, symbol Memory_EEPROM:93LCxxBxxOT
- added Y3: 12MHz, Crystal:Crystal_SMD_2520-4Pin_2.5x2.0mm, symbol Device:Crystal_GND24_Small
Connections:
- net +3V3: now also C10.1, C15.1, C19.1, C20.1, C21.1, C9.1, FB1.1, FB2.1, R19.1, R20.1, U3.16 (VCCIO), U3.36 (VCCIO), U3.44 (VREGIN), U3.50 (VCCIO), U6.6 (VCC)
- net GND: now also C10.2, C11.2, C12.2, C13.2, C14.2, C15.2, C16.2, C17.2, C18.2, C19.2, C20.2, C21.2, C22.2, C23.2, C9.2, J10.5 (Pin_5), J10.6 (Pin_6), J9.5 (Pin_5), J9.6 (Pin_6), R17.2, U3.10 (TEST), U3.21 (GND), U3.41 (GND), U3.45 (GND), U3.57 (GND), U6.2 (GND), Y3.2 (G), Y3.4 (G)
- net USB.D+: now also U3.8 (DP)
- net USB.D-: now also U3.7 (DM)
- new net: R18.1, R20.2, U6.1 (DO)
- new net: C16.1, R21.1, U3.3 (OSCI), Y3.1
- new net: C17.1, R21.2, U3.4 (OSCO), Y3.3
- new net: R17.1, U3.6 (REF)
- new net: R19.2, U3.11 (~{RESET})
- new net ADBUS0: J9.1 (Pin_1), U3.12 (ADBUS0)
- new net ADBUS1: J9.2 (Pin_2), U3.13 (ADBUS1)
- new net ADBUS2: J9.3 (Pin_3), U3.14 (ADBUS2)
- new net ADBUS3: J9.4 (Pin_4), U3.15 (ADBUS3)
- new net ADBUS4: J9.7 (Pin_7), U3.17 (ADBUS4)
- new net ADBUS5: J9.8 (Pin_8), U3.18 (ADBUS5)
- new net ADBUS6: J9.9 (Pin_9), U3.19 (ADBUS6)
- new net ADBUS7: J9.10 (Pin_10), U3.20 (ADBUS7)
- new net BDBUS0: J10.1 (Pin_1), U3.32 (BDBUS0)
- new net BDBUS1: J10.2 (Pin_2), U3.33 (BDBUS1)
- new net BDBUS2: J10.3 (Pin_3), U3.34 (BDBUS2)
- new net BDBUS3: J10.4 (Pin_4), U3.35 (BDBUS3)
- new net BDBUS4: J10.7 (Pin_7), U3.37 (BDBUS4)
- new net BDBUS5: J10.8 (Pin_8), U3.38 (BDBUS5)
- new net BDBUS6: J10.9 (Pin_9), U3.39 (BDBUS6)
- new net BDBUS7: J10.10 (Pin_10), U3.40 (BDBUS7)
- new net EECLK: U3.56 (EECLK), U6.4 (CLK)
- new net EECS: U3.1 (EECS), U6.5 (CS)
- new net EEDATA: R18.2, U3.55 (EEDATA), U6.3 (DI)
- new net VCORE: C18.1, C22.1, C23.1, U3.2 (VCORE), U3.31 (VCORE), U3.43 (VREGOUT)
- new net VPHY: C13.1, C14.1, FB2.2, U3.5 (VPHY)
- new net VPLL: C11.1, C12.1, FB1.2, U3.9 (VPLL)
- no-connect marks 0 -> 18
Other:
- moved on the sheet: D9

Commit message: Add 3x channels of spare LEDs for general breadboard use, add silkscreen.  Ordered this version
Parts:
- C11, C14, C15, C19, C20, C21, C22, C23, C9: JLCPCB Part No. (none) -> C77020; MPN (none) -> GRM155R71H104KE14D
- C16, C17: JLCPCB Part No. (none) -> C106201; MPN (none) -> CC0402JRNPO9BN120
- FB1, FB2: JLCPCB Part No. (none) -> C76891; MPN (none) -> BLM15PD121SN1D
- J10, J9: FT Rotation Offset (none) -> 90; JLCPCB Part No. (none) -> C492422; MPN (none) -> PZ254V-12-10P
- R17, R19: JLCPCB Part No. (none) -> C114760; MPN (none) -> RC0402FR-0712KL
- R18: JLCPCB Part No. (none) -> C60488; MPN (none) -> RC0402FR-072KL
- R20: JLCPCB Part No. (none) -> C60490; MPN (none) -> RC0402FR-0710KL
- R21: JLCPCB Part No. (none) -> C138033; MPN (none) -> RC0402FR-071ML
- U3: FT Rotation Offset (none) -> -90; JLCPCB Part No. (none) -> C3227935
- U6: value 93LCxxBxxOT -> 93LC56BxxOT; JLCPCB Part No. (none) -> C190271; MPN (none) -> 93LC56BT-I/OT
Other:
- company: (none) -> SK Electronics Consulting LLC
- title: (none) -> USB 2.0 Hub for Gridifinity
