File: Gridfinity-USB-hub/downstream_port_with_sensor.kicad_sch (KiCad schematic)
At the start: 13 parts, among them J7 USB_C_Receptacle_USB2.0_16P, U7 INA226

Commit message: Add 3x channels of spare LEDs for general breadboard use, add silkscreen.  Ordered this version
Parts:
- C26, C28, C30: JLCPCB Part No. (none) -> C77020; MPN (none) -> GRM155R71H104KE14D
- R22, R23: JLCPCB Part No. (none) -> C60490; MPN (none) -> RC0402FR-0710KL
- R28: JLCPCB Part No. C844909 -> C2988648; MPN WSLP12065L000FEA -> HoLLR1206-1W-5mR-1%
- U7: JLCPCB Part No. (none) -> C49851; MPN (none) -> INA226AIDGSR
Other:
- company: (none) -> SK Electronics Consulting LLC
- title: (none) -> USB 2.0 Hub for Gridifinity
Changed lines of the file:
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@@
 	(generator_version "9.0")
 	(paper "A4")
+	(title_block
+		(title "USB 2.0 Hub for Gridifinity")
+		(date "2026-02-16")
+		(rev "2")
+		(company "SK Electronics Consulting LLC")
+	)
 	(text "Future Feature Ideas:\n1. Add a power monitor to each channel\n2. Jumpers to adjust R_{p} values\n"
 		(exclude_from_sim no)
@@
 			)
 		)
+		(property "JLCPCB Part No." "C49851"
+			(at 76.2 76.2 0)
+			(effects
+				(font
+					(size 1.27 1.27)
+				)
+				(hide yes)
+			)
+		)
+		(property "MPN" "INA226AIDGSR"
+			(at 76.2 76.2 0)
+			(effects
+				(font
+					(size 1.27 1.27)
+				)
+				(hide yes)
+			)
+		)
 		(pin "4"
 		)
@@
 			)
 		)
-		(property "JLCPCB Part No." ""
+		(property "JLCPCB Part No." "C60490"
 			(at 151.13 82.55 0)
 			(effects
@@
 		)
 		(property "KLC_S4.2_VREGOUT" ""
+			(at 151.13 82.55 0)
+			(effects
+				(font
+					(size 1.27 1.27)
+				)
+				(hide yes)
+			)
+		)
+		(property "MPN" "RC0402FR-0710KL"
 			(at 151.13 82.55 0)
 			(effects
@@
 			)
 		)
-		(property "MPN" "WSLP12065L000FEA"
+		(property "MPN" "HoLLR1206-1W-5mR-1%"
 			(at 110.49 39.37 90)
 			(effects
@@
 			)
 		)
-		(property "JLCPCB Part No." "C844909"
+		(property "JLCPCB Part No." "C2988648"
 			(at 110.49 39.37 0)
 			(effects
@@
 			)
 		)
-		(property "JLCPCB Part No." ""
+		(property "JLCPCB Part No." "C77020"
 			(at 110.49 72.39 0)
 			(effects
@@
 			)
 		)
-		(property "MPN" ""
+		(property "MPN" "GRM155R71H104KE14D"
 			(at 110.49 72.39 0)
 			(effects
@@
 			)
 		)
-		(property "MPN" ""
+		(property "MPN" "GRM155R71H104KE14D"
 			(at 68.58 62.23 0)
 			(effects
@@
 			)
 		)
-		(property "JLCPCB Part No." ""
+		(property "JLCPCB Part No." "C77020"
 			(at 68.58 62.23 90)
 			(effects
@@
 			)
 		)
-		(property "JLCPCB Part No." ""
+		(property "JLCPCB Part No." "C60490"
 			(at 158.75 82.55 0)
 			(effects
@@
 		)
 		(property "KLC_S4.2_VREGOUT" ""
+			(at 158.75 82.55 0)
+			(effects
+				(font
+					(size 1.27 1.27)
+				)
+				(hide yes)
+			)
+		)
+		(property "MPN" "RC0402FR-0710KL"
 			(at 158.75 82.55 0)
 			(effects
@@
 			)
 		)
-		(property "JLCPCB Part No." ""
+		(property "JLCPCB Part No." "C77020"
 			(at 93.98 66.04 0)
 			(effects
@@
 			)
 		)
-		(property "MPN" ""
+		(property "MPN" "GRM155R71H104KE14D"
 			(at 93.98 66.04 0)
 			(effects
