File: Gridfinity-USB-hub/upstream.kicad_sch (KiCad schematic)
At the start: 5 parts, among them J3 USB_C_Receptacle_USB2.0_16P

Commit message: Checkpoint, changing computers
Parts:
- removed C3: 47u, Capacitor_SMD:C_1206_3216Metric, symbol Device:C_Small
- removed D2: Green, LED_SMD:LED_0402_1005Metric, symbol Device:LED_Small
- removed J3: USB_C_Receptacle_USB2.0_16P, Connector_USB:USB_C_Receptacle_G-Switch_GT-USB-7051x, symbol Connector:USB_C_Receptacle_USB2.0_16P
- removed R6, R7: 56k, Resistor_SMD:R_0402_1005Metric, symbol Device:R_Small
- added J1: USB_C_Receptacle_USB2.0_16P, Connector_USB:USB_C_Receptacle_G-Switch_GT-USB-7051x, symbol Connector:USB_C_Receptacle_USB2.0_16P
- added R1, R2: 5.1k, Resistor_SMD:R_0402_1005Metric, symbol Device:R_Small
- added TH1: 6V/2A, Resistor_SMD:R_0603_1608Metric, symbol Device:Thermistor_PTC
Connections:
- net +5V: now also TH1.2
- net GND: now also J1.A1 (GND), J1.A12 (GND), J1.B1 (GND), J1.B12 (GND), J1.S1 (SHIELD), R1.2, R2.2
- new net CC1: J1.A5 (CC1), R2.1
- new net CC2: J1.B5 (CC2), R1.1
- new net Upstream.D+: J1.A6 (D+), J1.B6 (D+)
- new net Upstream.D-: J1.A7 (D-), J1.B7 (D-)
- new net VBUS: J1.A4 (VBUS), J1.A9 (VBUS), J1.B4 (VBUS), J1.B9 (VBUS), TH1.1
Other:
- note removed: "Future Feature Ideas: 1. Add a power monitor to each channel 2. Jumpers to adjust R_{p} values"

Commit message: V2 complete, ready for review and polish
Parts:
- removed TH1: 6V/2A, Resistor_SMD:R_0603_1608Metric, symbol Device:Thermistor_PTC
Connections:
- net GND: now also J1.SH (SHIELD); no longer J1.S1 (SHIELD)

Commit message: Add 3x channels of spare LEDs for general breadboard use, add silkscreen.  Ordered this version
Other:
- company: (none) -> SK Electronics Consulting LLC
- title: (none) -> USB 2.0 Hub for Gridifinity
Changed lines of the file:
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@@
 	(generator_version "9.0")
 	(paper "A4")
+	(title_block
+		(title "USB 2.0 Hub for Gridifinity")
+		(date "2026-02-16")
+		(rev "2")
+		(company "SK Electronics Consulting LLC")
+	)
 	(junction
 		(at 100.33 53.34)
