File: pixelblaze_battery_backpack/charger.kicad_sch (KiCad schematic)
At the start: 22 parts, among them J1 Conn_01x01, J2 Conn_01x01, J3 Conn_01x01, J4 Conn_01x01, U3 BQ25798

Commit message: Finalized V2.
Parts:
- added C37: 1n, Capacitor_SMD:C_0402_1005Metric, symbol Device:C_Small
- J1, J2, J3, J4: footprint Battery:BatteryClip_MYoung_MY-18650-01 -> Battery:BatteryClip_Keystone_54_D16-19mm
Connections:
- net BATT+: now also C37.1
- net at U3.24 (SDRV): now also C37.2
- no-connect marks 3 -> 2
Other:
- note removed: "${ERC_ERROR SDRV Cap}Add 1nF cap to SDRV Pin"
- moved on the sheet: C1, C2, C3, J1, J2, J3, J4, R8
