File: pixelblaze_battery_backpack/usb_input.kicad_sch (KiCad schematic)
At the start: 4 parts, among them J5 USB_C_Receptacle_USB2.0_16P, U1 HUSB238

Commit message: Finalized V2.
Parts:
- U1: FT Rotation Offset (none) -> -90
Connections:
- net GND: now also J5.SH (SHIELD); no longer J5.S1 (SHIELD)
Changed lines of the file:
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@@
 			)
 		)
-		(property "FT Rotation Offset" ""
+		(property "FT Rotation Offset" "-90"
 			(at 156.21 83.82 0)
 			(effects
@@
 		(pin "B5"
 		)
-		(pin "S1"
+		(pin "SH"
 		)
 		(pin "B7"
